File: Hardware/PCB/PacSat_Dev_RevD_240223/Power_Divider.kicad_sch (KiCad schematic)
At the start: 38 parts, among them P601 U_FL, Q601 SAV-331+, T601 ADT4-1WT+, U602 LT6657AHMS8-2.5, U604 RBP-140+

Commit message: Updated PacSat Rev D files under Hardware PCB
Connections:
- net GND: now also T601.3 (AB), T601.5 (SC); no longer T601.2 (AB), T601.4 (SC)
- net S+: now also T601.6 (SB); no longer T601.5 (SB)
- net S-: now also T601.4 (SA); no longer T601.3 (SA)
- no-connect marks 2 -> 3
